File: pcb/mainboard.sch (EAGLE design)
At the start: 129 parts, among them IC1 STM32F401CCU6, IC11 CP2102, IC2 S25FL064K, IC3 LM3671MF-ADJ, IC4 AX5243, IC5 M66, IC6 NCP1521BMU, IC7 24LC256SN, IC8 TPS54061, IC9 LTC4413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

Commit message: Add a to-do list for the next board revision
Other:
- note added: "add cap to ground to the NRST line"
- note added: "bump major version"
- note added: "remove 60V power supply"
- note added: "remove I2C EEPROM"
- note added: "remove I2C connector"
- note added: "replace AX5243 radio with SX1231"
- note removed: "add PTC to VIN"
- note removed: "replace VIN sensing resistor (bigger package)"
Changed lines of the file:
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@@
 <wire x1="261.62" y1="332.74" x2="261.62" y2="383.54" width="1.016" layer="109"/>
 <text x="-121.92" y="-25.4" size="1.778" layer="108">move the console USART to PA9/PA10 to enable bootloader over USART</text>
-<text x="-121.92" y="-27.94" size="1.778" layer="108">add PTC to VIN</text>
-<text x="-121.92" y="-30.48" size="1.778" layer="108">replace VIN sensing resistor (bigger package)</text>
-<text x="-121.92" y="-33.02" size="1.778" layer="108">replace NCP1521</text>
+<text x="-121.92" y="-27.94" size="1.778" layer="108">replace NCP1521</text>
 <text x="12.7" y="378.46" size="1.778" layer="97">UXB bus output power OR</text>
 <text x="121.92" y="378.46" size="1.778" layer="97">Main power supply</text>
@@
 <text x="27.94" y="-17.78" size="1.778" layer="97">unodex-connect-42-0.1.0</text>
 <text x="27.94" y="-22.86" size="1.778" layer="97">(c) 2017, qyx@krtko.org, CC-BY-SA</text>
+<text x="-121.92" y="-30.48" size="1.778" layer="108">add cap to ground to the NRST line</text>
+<text x="-121.92" y="-33.02" size="1.778" layer="108">remove 60V power supply</text>
+<text x="-121.92" y="-35.56" size="1.778" layer="108">replace AX5243 radio with SX1231</text>
+<text x="-121.92" y="-38.1" size="1.778" layer="108">remove I2C connector</text>
+<text x="-121.92" y="-40.64" size="1.778" layer="108">remove I2C EEPROM</text>
+<text x="-121.92" y="-43.18" size="1.778" layer="108">bump major version</text>
 </plain>
 <instances>
